File: ESP32-Tayloe-Mixer.kicad_pcb (KiCad board)
At the start: 2 copper layers, 116.3 x 79.9 mm, 63 parts, among them J1 Jack-DC, J2 BNC, J3 Audio_Jack, J4 Conn_01x03, T1 T50_SPLITTER, U1 LM358, U2 LM358, U201 ESP32-15-PIN, U202 PCBARTISTS-ES8388, U203 si5351, U3 AMS1117, U6 MCP1703A-2502_SOT223, U8 FST3253

Commit message: Update ESP32-Tayloe-Mixer.kicad_pcb
Parts:
- moved U201 3.29 mm to (147.0, 101.1)
- moved U202 0.11 mm to (117.4, 132.8)
