File: ESP32-Tayloe-Mixer.sch (KiCad schematic (older format))
At the start: 63 parts, among them J1 Jack-DC, J2 BNC, J3 Audio_Jack, J4 Conn_01x03, T1 T50_SPLITTER, U1 LM358, U2 LM358, U201 ESP32-15-PIN, U202 PCBARTISTS-ES8388, U203 si5351, U3 AMS1117, U6 MCP1703A-2502_SOT223, U8 FST3253

Commit message: fixed schematic
Parts:
- L1: value Inductor -> T30-6 22T
- T1: value T50_SPLITTER -> T30-6 11T:11T:22T
Changed lines of the file:
@@
 P 17350 10650
 F 0 "T1" H 17350 9400 50  0000 C CNN
-F 1 "T50_SPLITTER" H 17350 10550 50  0000 C CNN
+F 1 "T30-6 11T:11T:22T" H 17350 10550 50  0000 C CNN
 F 2 "Xenir:T50 Trifilar" H 17350 10650 50  0001 C CNN
 F 3 "" H 17350 10650 50  0001 C CNN
@@
 P 18700 9650
 F 0 "L1" H 18700 9600 50  0000 C CNN
-F 1 "Inductor" H 18700 9750 50  0000 C CNN
+F 1 "T30-6 22T" H 18700 9750 50  0000 C CNN
 F 2 "Xenir:T37_Inductor" H 18700 9750 50  0001 C CNN
 F 3 "" H 18700 9750 50  0001 C CNN

Commit message: gg
Parts:
- C1, C12, C13, C17, C19, C2, C203, C204, C22, C23, C24, C25, C30, C4, C5, C7, C78: symbol Xenir:Capacitor -> ESP32-Tayloe-Mixer-rescue:Capacitor-Xenir
- C11, C14, C16, C18, C79: symbol Xenir:Cap_Polarized -> ESP32-Tayloe-Mixer-rescue:Cap_Polarized-Xenir
- J2: symbol Xenir:BNC -> ESP32-Tayloe-Mixer-rescue:BNC-Xenir
- J3: symbol Xenir:Audio_Jack -> ESP32-Tayloe-Mixer-rescue:Audio_Jack-Xenir
- L1: symbol Xenir:Inductor -> ESP32-Tayloe-Mixer-rescue:Inductor-Xenir
- R1, R11, R12, R13, R14, R147, R148, R15, R16, R17, R18, R19, R2, R20, R201, R202, R3, R4, R5, R6, R7: symbol Xenir:Resistor -> ESP32-Tayloe-Mixer-rescue:Resistor-Xenir
- T1: symbol Xenir:T50_SPLITTER -> ESP32-Tayloe-Mixer-rescue:T50_SPLITTER-Xenir
- U1, U2: symbol Xenir:LM358 -> ESP32-Tayloe-Mixer-rescue:LM358-Xenir
- U201: symbol Xenir:ESP32-15-PIN -> ESP32-Tayloe-Mixer-rescue:ESP32-15-PIN-Xenir
- U202: symbol Xenir:PCBARTISTS-ES8388 -> ESP32-Tayloe-Mixer-rescue:PCBARTISTS-ES8388-Xenir
- U203: symbol Xenir:si5351 -> ESP32-Tayloe-Mixer-rescue:si5351-Xenir
- U8: symbol Xenir:FST3253 -> ESP32-Tayloe-Mixer-rescue:FST3253-Xenir
- VR1: symbol Xenir:Trimpot -> ESP32-Tayloe-Mixer-rescue:Trimpot-Xenir
Changed lines of the file:
@@
 	16650 13600 16650 12700
 $Comp
-L Xenir:Capacitor C30
+L ESP32-Tayloe-Mixer-rescue:Capacitor-Xenir C30
 U 1 1 5EE9C731
 P 17750 11350
@@
 	12850 11700 12850 11300
 $Comp
-L Xenir:Resistor R1
+L ESP32-Tayloe-Mixer-rescue:Resistor-Xenir R1
 U 1 1 5EF82F89
 P 10450 11300
@@
 $EndComp
 $Comp
-L Xenir:Resistor R3
+L ESP32-Tayloe-Mixer-rescue:Resistor-Xenir R3
 U 1 1 5EF82F8F
 P 10850 11700
@@
 $EndComp
 $Comp
-L Xenir:Resistor R11
+L ESP32-Tayloe-Mixer-rescue:Resistor-Xenir R11
 U 1 1 5EF82F95
 P 12650 11300
@@
 $EndComp
 $Comp
-L Xenir:Resistor R13
+L ESP32-Tayloe-Mixer-rescue:Resistor-Xenir R13
 U 1 1 5EF82F9B
 P 13050 11700
@@
 $EndComp
 $Comp
-L Xenir:Resistor R2
+L ESP32-Tayloe-Mixer-rescue:Resistor-Xenir R2
 U 1 1 5EF82FC5
 P 10450 12800
@@
 $EndComp
 $Comp
-L Xenir:Resistor R4
+L ESP32-Tayloe-Mixer-rescue:Resistor-Xenir R4
 U 1 1 5EF82FCB
 P 10850 13200
@@
 $EndComp
 $Comp
-L Xenir:Resistor R12
+L ESP32-Tayloe-Mixer-rescue:Resistor-Xenir R12
 U 1 1 5EF82FD1
 P 12650 12800
@@
 $EndComp
 $Comp
-L Xenir:Resistor R14
+L ESP32-Tayloe-Mixer-rescue:Resistor-Xenir R14
 U 1 1 5EF82FD7
 P 13050 13200
@@
 	17050 12200 17050 12400
 $Comp
-L Xenir:FST3253 U8
+L ESP32-Tayloe-Mixer-rescue:FST3253-Xenir U8
 U 1 1 6E1B97F5
 P 18200 11050
@@
 	16800 11800 17050 11800
 $Comp
-L Xenir:Resistor R17
+L ESP32-Tayloe-Mixer-rescue:Resistor-Xenir R17
 U 1 1 5EEBB81B
 P 15200 11950
@@
 $EndComp
 $Comp
-L Xenir:Resistor R18
+L ESP32-Tayloe-Mixer-rescue:Resistor-Xenir R18
 U 1 1 5EEBC201
 P 15200 12400
@@
 $EndComp
 $Comp
-L Xenir:Resistor R19
+L ESP32-Tayloe-Mixer-rescue:Resistor-Xenir R19
 U 1 1 5EEBC4DE
 P 15200 12850
@@
 $EndComp
 $Comp
-L Xenir:Resistor R20
+L ESP32-Tayloe-Mixer-rescue:Resistor-Xenir R20
 U 1 1 5EEBCADD
 P 15200 13300
@@
 $EndComp
 $Comp
-L Xenir:Capacitor C22
+L ESP32-Tayloe-Mixer-rescue:Capacitor-Xenir C22
 U 1 1 5EEBD3D7
 P 15400 12100
@@
 $EndComp
 $Comp
-L Xenir:Capacitor C23
+L ESP32-Tayloe-Mixer-rescue:Capacitor-Xenir C23
 U 1 1 5EEBE874
 P 15400 12550
@@
 $EndComp
 $Comp
-L Xenir:Capacitor C24
+L ESP32-Tayloe-Mixer-rescue:Capacitor-Xenir C24
 U 1 1 5EED34B4
 P 15400 13000
@@
 $EndComp
 $Comp
-L Xenir:Capacitor C25
+L ESP32-Tayloe-Mixer-rescue:Capacitor-Xenir C25
 U 1 1 5EED8105
 P 15400 13450
@@
 270
 $Comp
-L Xenir:LM358 U1
+L ESP32-Tayloe-Mixer-rescue:LM358-Xenir U1
 U 3 1 5EAF812F
 P 6200 1750
@@
 $EndComp
 $Comp
-L Xenir:LM358 U2
+L ESP32-Tayloe-Mixer-rescue:LM358-Xenir U2
 U 3 1 5EB0186E
 P 6650 1750
@@
 $EndComp
 $Comp
-L Xenir:Capacitor C12
+L ESP32-Tayloe-Mixer-rescue:Capacitor-Xenir C12
 U 1 1 5EB751C3
 P 8200 1750
@@
 	5750 1450 6100 1450
 $Comp
-L Xenir:LM358 U1
+L ESP32-Tayloe-Mixer-rescue:LM358-Xenir U1
 U 2 1 5F197569
 P 13150 11200
@@
 Connection ~ 13450 11200
 $Comp
-L Xenir:LM358 U2
+L ESP32-Tayloe-Mixer-rescue:LM358-Xenir U2
 U 2 1 5F1992ED
 P 13150 12700
@@
 Connection ~ 6550 1450
 $Comp
-L Xenir:Capacitor C13
+L ESP32-Tayloe-Mixer-rescue:Capacitor-Xenir C13
 U 1 1 5F243F69
 P 8550 1750
@@
 Connection ~ 10650 11300
 $Comp
-L Xenir:LM358 U2
+L ESP32-Tayloe-Mixer-rescue:LM358-Xenir U2
 U 1 1 5F344BC8
 P 10950 12700
@@
 Connection ~ 10650 12800
 $Comp
-L Xenir:LM358 U1
+L ESP32-Tayloe-Mixer-rescue:LM358-Xenir U1
 U 1 1 5F334557
 P 10950 11200
@@
 $EndComp
 $Comp
-L Xenir:si5351 U203
+L ESP32-Tayloe-Mixer-rescue:si5351-Xenir U203
 U 1 1 5E9EA10D
 P 16650 5500
@@
 	5750 1650 5750 2050
 $Comp
-L Xenir:Capacitor C1
+L ESP32-Tayloe-Mixer-rescue:Capacitor-Xenir C1
 U 1 1 6104EF39
 P 10100 11300
@@
 $EndComp
 $Comp
-L Xenir:Capacitor C2
+L ESP32-Tayloe-Mixer-rescue:Capacitor-Xenir C2
 U 1 1 610508A9
 P 10100 12800
@@
 LO_90
 $Comp
-L Xenir:T50_SPLITTER T1
+L ESP32-Tayloe-Mixer-rescue:T50_SPLITTER-Xenir T1
 U 1 1 60EFEA4B
 P 17350 10650
@@
 $EndComp
 $Comp
-L Xenir:Resistor R148
+L ESP32-Tayloe-Mixer-rescue:Resistor-Xenir R148
 U 1 1 60FC36BE
 P 16800 11150
@@
 $EndComp
 $Comp
-L Xenir:Resistor R147
+L ESP32-Tayloe-Mixer-rescue:Resistor-Xenir R147
 U 1 1 60FC45B4
 P 16550 11150
@@
 $EndComp
 $Comp
-L Xenir:Cap_Polarized C11
+L ESP32-Tayloe-Mixer-rescue:Cap_Polarized-Xenir C11
 U 1 1 61126761
 P 1400 1750
@@
 	2900 1600 3000 1600
 $Comp
-L Xenir:Cap_Polarized C14
+L ESP32-Tayloe-Mixer-rescue:Cap_Polarized-Xenir C14
 U 1 1 61126762
 P 3100 1750
@@
 Connection ~ 3000 1600
 $Comp
-L Xenir:BNC J2
+L ESP32-Tayloe-Mixer-rescue:BNC-Xenir J2
 U 1 1 5F509493
 P 21050 9950
@@
 $EndComp
 $Comp
-L Xenir:Cap_Polarized C16
+L ESP32-Tayloe-Mixer-rescue:Cap_Polarized-Xenir C16
 U 1 1 610A03F4
 P 2050 1750
@@
 $EndComp
 $Comp
-L Xenir:Capacitor C17
+L ESP32-Tayloe-Mixer-rescue:Capacitor-Xenir C17
 U 1 1 613E4B97
 P 2250 1750
@@
 $EndComp
 $Comp
-L Xenir:Resistor R15
+L ESP32-Tayloe-Mixer-rescue:Resistor-Xenir R15
 U 1 1 613DBAD6
 P 3700 1800
@@
 Connection ~ 3700 1600
 $Comp
-L Xenir:Resistor R16
+L ESP32-Tayloe-Mixer-rescue:Resistor-Xenir R16
 U 1 1 613DCC79
 P 3700 2400
@@
 $EndComp
 $Comp
-L Xenir:Cap_Polarized C18
+L ESP32-Tayloe-Mixer-rescue:Cap_Polarized-Xenir C18
 U 1 1 613DDE0F
 P 3500 2350
@@
 $EndComp
 $Comp
-L Xenir:Capacitor C19
+L ESP32-Tayloe-Mixer-rescue:Capacitor-Xenir C19
 U 1 1 613DE98D
 P 4000 2350
@@
 $EndComp
 $Comp
-L Xenir:Resistor R5
+L ESP32-Tayloe-Mixer-rescue:Resistor-Xenir R5
 U 1 1 612306CF
 P 15700 9550
@@
 $EndComp
 $Comp
-L Xenir:Resistor R6
+L ESP32-Tayloe-Mixer-rescue:Resistor-Xenir R6
 U 1 1 612306DA
 P 15700 10150
@@
 $EndComp
 $Comp
-L Xenir:Capacitor C4
+L ESP32-Tayloe-Mixer-rescue:Capacitor-Xenir C4
 U 1 1 612306EE
 P 16000 10100
@@
 Connection ~ 16000 9950
 $Comp
-L Xenir:Capacitor C5
+L ESP32-Tayloe-Mixer-rescue:Capacitor-Xenir C5
 U 1 1 613306E3
 P 18050 9900
@@
 Connection ~ 17700 10250
 $Comp
-L Xenir:Inductor L1
+L ESP32-Tayloe-Mixer-rescue:Inductor-Xenir L1
 U 1 1 6133F735
 P 18700 9650
@@
 $EndComp
 $Comp
-L Xenir:Capacitor C7
+L ESP32-Tayloe-Mixer-rescue:Capacitor-Xenir C7
 U 1 1 61340140
 P 19250 9650
@@
 $EndComp
 $Comp
-L Xenir:Resistor R7
+L ESP32-Tayloe-Mixer-rescue:Resistor-Xenir R7
 U 1 1 613406A2
 P 19600 9950
@@
 Connection ~ 1300 1600
 $Comp
-L Xenir:PCBARTISTS-ES8388 U202
+L ESP32-Tayloe-Mixer-rescue:PCBARTISTS-ES8388-Xenir U202
 U 1 1 6126113C
 P 18050 3950
@@
 $EndComp
 $Comp
-L Xenir:ESP32-15-PIN U201
+L ESP32-Tayloe-Mixer-rescue:ESP32-15-PIN-Xenir U201
 U 1 1 61262009
 P 14900 3950
@@
 $EndComp
 $Comp
-L Xenir:Capacitor C78
+L ESP32-Tayloe-Mixer-rescue:Capacitor-Xenir C78
 U 1 1 612A288A
 P 3450 3550
@@
 $EndComp
 $Comp
-L Xenir:Cap_Polarized C79
+L ESP32-Tayloe-Mixer-rescue:Cap_Polarized-Xenir C79
 U 1 1 612A2CBF
 P 3900 3550
@@
 Connection ~ 3800 3400
 $Comp
-L Xenir:Audio_Jack J3
+L ESP32-Tayloe-Mixer-rescue:Audio_Jack-Xenir J3
 U 1 1 612B3944
 P 21050 4600
@@
 	19950 3950 18850 3950
 $Comp
-L Xenir:Capacitor C203
+L ESP32-Tayloe-Mixer-rescue:Capacitor-Xenir C203
 U 1 1 612B729F
 P 19550 2850
@@
 $EndComp
 $Comp
-L Xenir:Resistor R201
+L ESP32-Tayloe-Mixer-rescue:Resistor-Xenir R201
 U 1 1 612B846F
 P 19350 2700
@@
 $EndComp
 $Comp
-L Xenir:Capacitor C204
+L ESP32-Tayloe-Mixer-rescue:Capacitor-Xenir C204
 U 1 1 612C0A2F
 P 20200 3150
@@
 $EndComp
 $Comp
-L Xenir:Resistor R202
+L ESP32-Tayloe-Mixer-rescue:Resistor-Xenir R202
 U 1 1 612C0A39
 P 20000 3000
@@
 $EndComp
 $Comp
-L Xenir:Trimpot VR1
+L ESP32-Tayloe-Mixer-rescue:Trimpot-Xenir VR1
 U 1 1 612E7453
 P 13000 3450
